Commit message: 

File: src/ugv_main/ugv_description/urdf/ugv_rover.urdf (robot description, URDF)
Before this commit: robot ugv_rover, 13 links, 12 joints
Joints:
- joint base_lidar_link_joint: origin xyz=0.0398145505519817 0 0.04 rpy=0 0 1.5708 -> xyz=0.0398145505519817 0 0.04 rpy=0 0 -1.5708

Commit message: 

File: src/ugv_main/ugv_description/urdf/ugv_rover.urdf (robot description, URDF)
Before this commit: robot ugv_rover, 13 links, 12 joints
Joints:
- joint base_lidar_link_joint: origin xyz=0.0398145505519817 0 0.04 rpy=0 0 -1.5708 -> xyz=0.0398145505519817 0 0.04 rpy=0 0 0

Commit message: 

File: src/ugv_main/ugv_description/urdf/ugv_rover.urdf (robot description, URDF)
Before this commit: robot ugv_rover, 13 links, 12 joints
Joints:
- joint base_lidar_link_joint: origin xyz=0.0398145505519817 0 0.04 rpy=0 0 0 -> xyz=0.0398145505519817 0 0.04 rpy=0 0 1.5708
